File: PCB_Business_Card.kicad_pcb (KiCad board)
At the start: 2 copper layers, 88.9 x 50.8 mm, 9 parts, among them U1 NT3H1101W0FTTJ

Commit message: my edits
Parts:
- removed G*** (x2): LOGO, LOGO
Other:
- board text added: "+39 3202439256"
- board text added: "Fabio Ricci"
- board text added: "Technician"
- board text added: "fabio.ricci@iit.it"
- board text added: "riccifab"
- board text removed: "Electrical Engineer"
- board text removed: "PCB3D_BR_PCB_Business_Card"
- board text removed: "PCB3D_TL_PCB_Business_Card"
- board text removed: "Rahim Aziz"
- board text removed: "linkedin.com/in/rahim-aziz"
- board text removed: "raziz1.github.io"

Commit message: Updated idk
Other:
- board text removed: "Technician"
Changed lines of the file:
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@@
 		(layer "Edge.Cuts")
 	)
-	(gr_text "Technician\n"
+	(gr_text "\n"
 		(at 174 74.5 0)
 		(layer "F.SilkS")
